Commit message: after hip joints are replaced

File: Simulator/SimulationModel/Mercury_Model/mercury_srlib (copy).urdf (robot description, URDF)
Before this commit: robot mercury, 23 links, 22 joints
Links:
- link abduct_l: geometry visual mesh filename=meshes/color_abduction_L.dae scale=0.001 0.001 0.001
- link abduct_r: geometry visual mesh filename=meshes/color_abduction_R.dae scale=0.001 0.001 0.001
- link body: mass 9.0 -> 8.0; geometry visual mesh filename=meshes/color_torso.dae scale=0.001 0.001 0.001
- link lfoot: geometry collision box size=0.2 0.01 0.01; visual mesh filename=meshes/color_foot_L.dae scale=1 1 1
- link rfoot: geometry collision box size=0.2 0.01 0.01; visual mesh filename=meshes/color_foot_R.dae scale=1 1 1
- link shank_l: geometry visual mesh filename=meshes/color_shank_L.dae scale=0.001 0.001 0.001
- link shank_r: geometry visual mesh filename=meshes/color_shank_R.dae scale=0.001 0.001 0.001
- link thigh_l: mass 3.6 -> 3.2; geometry visual mesh filename=meshes/color_thigh_L.dae scale=0.001 0.001 0.001
- link thigh_r: mass 3.6 -> 3.2; geometry visual mesh filename=meshes/color_thigh_L.dae scale=0.001 0.001 0.001
Joints:
- joint abduct_l_to_thigh_l_j: origin xyz=0.0 -0.005 -0.03535 rpy=0.0 0 0.007 -> xyz=0.0 0.0 -0.03535 rpy=-0.017 0 0.01
- joint abduct_r_to_thigh_r_j: origin xyz=0.0 0.0 -0.03535 rpy=0.01 0.0 0.007 -> xyz=0.0 0.0 -0.03535 rpy=0.01 0.0 0.0
- joint ankle_l: origin xyz=0.0 -0.002 -0.47 rpy=0 0 0 -> xyz=0.0 -0.008 -0.47 rpy=0 0 0; type fixed -> continuous
- joint ankle_r: type fixed -> continuous
- joint fixed_bodyled1: origin xyz=0.077 0.144 0.3 rpy=0 0 0 -> xyz=0.077 0.142 0.3 rpy=0 0 0
- joint fixed_bodyled2: origin xyz=0.077 -0.144 0.3 rpy=0 0 0 -> xyz=0.077 -0.142 0.3 rpy=0 0 0
- joint thigh_l_to_knee_l_j: origin xyz=0.0181 0.00 -0.4575 rpy=0 0 0.005 -> xyz=0.0181 -0.005 -0.4575 rpy= 0.0 0 0.00
- joint thigh_r_to_knee_r_j: origin xyz=0.0181 0.00 -0.4575 rpy=0.0 0 0.0 -> xyz=0.0181 0.005 -0.4575 rpy=0.02 0 0.02

File: Simulator/SimulationModel/Mercury_Model/mercury_srlib.urdf (robot description, URDF)
Before this commit: robot mercury, 23 links, 22 joints
Links:
- link abduct_l: geometry 
- link abduct_r: geometry 
- link body: mass 8.0 -> 9.0; geometry 
- link lfoot: geometry 
- link rfoot: geometry 
- link shank_l: geometry 
- link shank_r: geometry 
- link thigh_l: mass 3.2 -> 3.6; geometry 
- link thigh_r: mass 3.2 -> 3.6; geometry 
Joints:
- joint abduct_l_to_thigh_l_j: origin xyz=0.0 0.0 -0.03535 rpy=-0.017 0 0.01 -> xyz=0.0 0.0 -0.03535 rpy=0.0 0 0.007
- joint abduct_r_to_thigh_r_j: origin xyz=0.0 0.0 -0.03535 rpy=0.01 0.0 0.0 -> xyz=0.0 0.0 -0.03535 rpy=0.01 0.0 0.007
- joint ankle_l: origin xyz=0.0 -0.008 -0.47 rpy=0 0 0 -> xyz=0.0 -0.002 -0.47 rpy=0 0 0
- joint fixed_bodyled1: origin xyz=0.077 0.142 0.3 rpy=0 0 0 -> xyz=0.077 0.144 0.3 rpy=0 0 0
- joint fixed_bodyled2: origin xyz=0.077 -0.142 0.3 rpy=0 0 0 -> xyz=0.077 -0.144 0.3 rpy=0 0 0
- joint fixed_led10: origin xyz=0.0 -0.033 -0.47 rpy=0 0 0 -> xyz=0.0 -0.033 -0.50 rpy=0 0 0
- joint fixed_led4: origin xyz=0.0 -0.025 -0.47 rpy=0 0 0 -> xyz=0.0 -0.025 -0.50 rpy=0 0 0
- joint fixed_led5: origin xyz=0.0 0.025 -0.47 rpy=0 0 0 -> xyz=0.0 0.025 -0.50 rpy=0 0 0
- joint fixed_led9: origin xyz=0.0 0.017 -0.47 rpy=0 0 0 -> xyz=0.0 0.017 -0.50 rpy=0 0 0
- joint thigh_l_to_knee_l_j: origin xyz=0.0181 -0.005 -0.4575 rpy= 0.0 0 0.00 -> xyz=0.0181 0.00 -0.4575 rpy=0 0 0
- joint thigh_r_to_knee_r_j: origin xyz=0.0181 0.005 -0.4575 rpy=0.02 0 0.02 -> xyz=0.0181 0.00 -0.4575 rpy=0.0 0 0.0
