Commit message: update simulation and added new robot valkyrie and atlas

File: Simulator/SimulationModel/Mercury_Model/mercury_srlib.urdf (robot description, URDF)
Before this commit: robot mercury, 23 links, 22 joints
Links:
- link abduct_l: geometry visual mesh filename=meshes/color_abduction_L.dae scale=0.001 0.001 0.001
- link abduct_r: geometry visual mesh filename=meshes/color_abduction_R.dae scale=0.001 0.001 0.001
- link body: geometry visual mesh filename=meshes/white_torso.obj scale=0.508 0.508 0.508
- link lfoot: geometry visual mesh filename=meshes/color_foot_L.obj scale=1 1 1
- link rfoot: geometry visual mesh filename=meshes/color_foot_R.obj scale=1 1 1
- link shank_l: geometry visual mesh filename=meshes/color_shank_L.dae scale=0.001 0.001 0.001
- link shank_r: geometry visual mesh filename=meshes/color_shank_R.dae scale=0.001 0.001 0.001
- link thigh_l: geometry visual mesh filename=meshes/color_thigh_L.dae scale=0.001 0.001 0.001
- link thigh_r: geometry visual mesh filename=meshes/color_thigh_R.dae scale=0.001 0.001 0.001

Commit message: walking with the previous controller in simulation

File: Simulator/SimulationModel/Mercury_Model/mercury_srlib.urdf (robot description, URDF)
Before this commit: robot mercury, 23 links, 22 joints
Joints:
- joint abduct_l_to_thigh_l_j: origin xyz=0.0 0.0 -0.03535 rpy=0.0 0 0.007 -> xyz=0.0 -0.005 -0.03535 rpy=0.0 0 0.007

Commit message: wblc dynamics control part is done

File: Simulator/SimulationModel/Mercury_Model/mercury_srlib.urdf (robot description, URDF)
Before this commit: robot mercury, 23 links, 22 joints
Joints:
- joint thigh_l_to_knee_l_j: origin xyz=0.0181 0.00 -0.4575 rpy=0 0 0 -> xyz=0.0181 0.00 -0.4575 rpy=0 0 0.005

Commit message: push_recovery experiment

File: Simulator/SimulationModel/Mercury_Model/mercury_srlib.urdf (robot description, URDF)
Before this commit: robot mercury, 23 links, 22 joints
Joints:
- joint ankle_l: origin xyz=0.0 -0.002 -0.47 rpy=0 0 0 -> xyz=0.005 -0.02 -0.47 rpy=0 0 0
- joint ankle_r: origin xyz=0.0 0.0 -0.47 rpy=0 0 0 -> xyz=0.005 -0.01 -0.47 rpy=0 0 0
- joint thigh_l_to_knee_l_j: origin xyz=0.0181 0.00 -0.4575 rpy=0 0 0.005 -> xyz=0.0181 -0.01 -0.4575 rpy=0 0 0.005
