Commit message: model modification of dracobip

File: RobotSystems/DracoBip/DracoBip.urdf (robot description, URDF)
Before this commit: robot Draco, 11 links, 10 joints
Joints:
- joint lHipYaw: origin xyz=-0.0222 0.0870 -0.2951 rpy=0 0 0 -> xyz=-0.0222 0.0870 0.0 rpy=0 0 0
- joint rHipYaw: origin xyz=-0.0222 -0.0870 -0.2951 rpy=0 0 0 -> xyz=-0.0222 -0.0870 0.0 rpy=0 0 0

File: Simulator/SimulationModel/DracoBip/DracoBip.urdf (robot description, URDF)
Before this commit: robot Draco, 11 links, 10 joints
Joints:
- joint lHipYaw: origin xyz=-0.0222 0.0870 -0.2951 rpy=0 0 0 -> xyz=-0.0222 0.0870 0.0 rpy=0 0 0
- joint rHipYaw: origin xyz=-0.0222 -0.0870 -0.2951 rpy=0 0 0 -> xyz=-0.0222 -0.0870 0.0 rpy=0 0 0
