Commit message: valkyrie hand pos and ori task test

File: Simulator/SimulationModel/Valkyrie/valkyrie_simple.urdf (robot description, URDF)
Before this commit: robot valkyrie, 76 links, 75 joints
Joints:
- joint leftIndexFingerPitch1: origin xyz=0.0022 0.0976 0.0235 rpy=0.1745 0.0 0.0 -> xyz=0.0022 0.0976 0.0235 rpy=0.1745 0.0 -0.1
- joint leftIndexFingerPitch2: origin xyz=0.0 0.0381 0.0 rpy=0.0 0.0 0.0 -> xyz=0.0 0.0381 0.0 rpy=0.0 0.0 -0.5
- joint leftThumbPitch1: origin xyz=0.0 0.0 0.0229 rpy=0.3491 0.0 0.0 -> xyz=0.0 0.0 0.0229 rpy=0.1491 0.0 0.0
- joint leftThumbPitch2: origin xyz=0.0 0.0066 0.0375 rpy=0.0 0.0 0.0 -> xyz=0.0 0.0066 0.0375 rpy=0. 0.0 0.0
- joint leftThumbPitch3: origin xyz=0.0 0.0049 0.0275 rpy=0.0 0.0 0.0 -> xyz=0.0 0.0049 0.0275 rpy=-0.5 0.0 0.0
- joint leftThumbRoll: origin xyz=0.0049 0.0351 0.0228 rpy=-0.3491 0.0 0.0 -> xyz=0.0049 0.0351 0.0228 rpy=-0.3491 1.3 0.0

Commit message: valkyrie is holding a paper cup

File: Simulator/SimulationModel/Valkyrie/valkyrie_simple.urdf (robot description, URDF)
Before this commit: robot valkyrie, 76 links, 75 joints
Links:
- added link leftCup, mass 0.000001; visual mesh filename=coffee_cup/coffee_cup.obj scale=0.014 0.014 0.014
Joints:
- added joint leftPalmCup: type fixed, parent leftPalm, child leftCup, origin xyz=0.06 0.11 -0.1 rpy=-1.57 0 0, axis 1 0 0, limit lower=-0.62 upper=0.625 effort=14 velocity=1
- joint leftIndexFingerPitch3: origin xyz=0.0 0.0229 0 rpy=0.0 0.0 0.0 -> xyz=0.0 0.0229 0 rpy=0.0 0.0 -0.6
- joint leftMiddleFingerPitch1: origin xyz=0.0022 0.097 -0.0119 rpy=-0.1222 0.0 0.0 -> xyz=0.0022 0.097 -0.0119 rpy=-0.1222 0.0 -0.2
- joint leftMiddleFingerPitch2: origin xyz=0.0 0.0381 0.0 rpy=0.0 0.0 0.0 -> xyz=0.0 0.0381 0.0 rpy=0.0 0.0 -0.5
- joint leftMiddleFingerPitch3: origin xyz=0.0 0.0229 0.0 rpy=0.0 0.0 0.0 -> xyz=0.0 0.0229 0.0 rpy=0.0 0.0 -0.5
- joint leftPinkyPitch1: origin xyz=0.0022 0.0838 -0.041 rpy=-0.1222 0.0 0.0 -> xyz=0.0022 0.0838 -0.041 rpy=-0.1222 0.0 -0.20
- joint leftPinkyPitch2: origin xyz=0.0 0.0381 0.0 rpy=0.0 0.0 0.0 -> xyz=0.0 0.0381 0.0 rpy=0.0 0.0 -0.45
- joint leftPinkyPitch3: origin xyz=0.0 0.0229 0.0 rpy=0.0 0.0 0.0 -> xyz=0.0 0.0229 0.0 rpy=0.0 0.0 -0.4
