Commit message: move to HCRL

File: RobotSystems/Mercury/mercury.urdf (robot description, URDF)
Before this commit: robot mercury, 21 links, 20 joints
Links:
- link body: mass 9.5 -> 8.0

Commit message: mercury right leg kinematics calibration is done

File: RobotSystems/Mercury/mercury.urdf (robot description, URDF)
Before this commit: robot mercury, 21 links, 20 joints
Links:
- added link lleg_led4, mass 0.000000000001
- added link rleg_led4, mass 0.000000000001
Joints:
- added joint fixed_led10: type fixed, parent shank_l, child lleg_led4, origin xyz=0.0 -0.025 -0.47 rpy=0 0 0, axis 0 1 0
- added joint fixed_led5: type fixed, parent shank_r, child rleg_led4, origin xyz=0.0 0.025 -0.47 rpy=0 0 0, axis 0 1 0
- joint abduct_r_to_thigh_r_j: origin xyz=0.0 0.0 -0.03535 rpy=0.015 0.0 -0.02 -> xyz=0.0 0.0 -0.03535 rpy=0.01 0.0 0.0
- joint fixed_led2: origin xyz=0.075 0.005 -0.42 rpy=0 0 0 -> xyz=0.075 0.0 -0.42 rpy=0 0 0
- joint fixed_led3: origin xyz=0.0 -0.02 -0.060 rpy=0 0 0 -> xyz=0.035 -0.0 -0.050 rpy=0 0 0
- joint fixed_led4: origin xyz=0.0 -0.0365 -0.47 rpy=0 0 0 -> xyz=0.0 -0.025 -0.47 rpy=0 0 0
- joint fixed_led7: origin xyz=0.075 -0.005 -0.42 rpy=0 0 0 -> xyz=0.075 0.0 -0.42 rpy=0 0 0
- joint fixed_led8: origin xyz=0.0 0.02 -0.062 rpy=0 0 0 -> xyz=0.035 0.0 -0.05 rpy=0 0 0
- joint fixed_led9: origin xyz=0.0 0.02 -0.47 rpy=0 0 0 -> xyz=0.0 0.025 -0.47 rpy=0 0 0
- joint thigh_r_to_knee_r_j: origin xyz=0.0181 0.005 -0.4575 rpy=0.02 0 0.04 -> xyz=0.0181 0.005 -0.4575 rpy=0.02 0 0.02

Commit message: left leg kinematics tune is done

File: RobotSystems/Mercury/mercury.urdf (robot description, URDF)
Before this commit: robot mercury, 23 links, 22 joints
Joints:
- joint abduct_l_to_thigh_l_j: origin xyz=0.0 0.0 -0.03535 rpy=0.0 0 0.01 -> xyz=0.0 0.0 -0.03535 rpy=-0.017 0 0.01
- joint ankle_l: origin xyz=0.0 -0.0165 -0.47 rpy=0 0 0 -> xyz=0.0 -0.008 -0.47 rpy=0 0 0
- joint fixed_led10: origin xyz=0.0 -0.025 -0.47 rpy=0 0 0 -> xyz=0.0 -0.033 -0.47 rpy=0 0 0
- joint fixed_led8: origin xyz=0.035 0.0 -0.05 rpy=0 0 0 -> xyz=0.04 0.0 -0.045 rpy=0 0 0
- joint fixed_led9: origin xyz=0.0 0.025 -0.47 rpy=0 0 0 -> xyz=0.0 0.017 -0.47 rpy=0 0 0
- joint thigh_l_to_knee_l_j: origin xyz=0.0181 -0.005 -0.4575 rpy= 0.008 0 0.00 -> xyz=0.0181 -0.005 -0.4575 rpy= 0.0 0 0.00

Commit message: 35 steps

File: RobotSystems/Mercury/mercury.urdf (robot description, URDF)
Before this commit: robot mercury, 23 links, 22 joints
Links:
- link abduct_l: geometry 
- link abduct_r: geometry 
- link body: mass 8.0 -> 9.0; geometry 
- link lfoot: geometry 
- link rfoot: geometry 
- link shank_l: geometry 
- link shank_r: geometry 
- link thigh_l: mass 3.2 -> 3.6; geometry 
- link thigh_r: mass 3.2 -> 3.6; geometry 
Joints:
- joint abduct_r_to_thigh_r_j: origin xyz=0.0 0.0 -0.03535 rpy=0.01 0.0 0.0 -> xyz=0.0 0.0 -0.03535 rpy=0.02 0.0 0.0
- joint thigh_l_to_knee_l_j: origin xyz=0.0181 -0.005 -0.4575 rpy= 0.0 0 0.00 -> xyz=0.0181 -0.005 -0.4575 rpy=0 0 0
- joint thigh_r_to_knee_r_j: origin xyz=0.0181 0.005 -0.4575 rpy=0.02 0 0.02 -> xyz=0.0181 0.005 -0.4575 rpy=0.0 0 0.02

Commit message: update before demo

File: RobotSystems/Mercury/mercury.urdf (robot description, URDF)
Before this commit: robot mercury, 23 links, 22 joints
Joints:
- joint ankle_l: origin xyz=0.0 -0.002 -0.47 rpy=0 0 0 -> xyz=0.035 -0.002 -0.47 rpy=0 0 0
- joint ankle_r: origin xyz=0.0 0.0 -0.47 rpy=0 0 0 -> xyz=0.035 0.0 -0.47 rpy=0 0 0

Commit message: just in case control pc

File: RobotSystems/Mercury/mercury.urdf (robot description, URDF)
Before this commit: robot mercury, 23 links, 22 joints
Joints:
- joint ankle_l: origin xyz=0.035 -0.002 -0.47 rpy=0 0 0 -> xyz=0.025 -0.002 -0.47 rpy=0 0 0
- joint ankle_r: origin xyz=0.035 0.0 -0.47 rpy=0 0 0 -> xyz=0.025 0.0 -0.47 rpy=0 0 0

Commit message: simulation based debugging

File: RobotSystems/Mercury/mercury.urdf (robot description, URDF)
Before this commit: robot mercury, 23 links, 22 joints
Joints:
- joint ankle_l: origin xyz=0.025 -0.002 -0.47 rpy=0 0 0 -> xyz=0.0 -0.002 -0.47 rpy=0 0 0
- joint ankle_r: origin xyz=0.025 0.0 -0.47 rpy=0 0 0 -> xyz=0.0 0.0 -0.47 rpy=0 0 0

Commit message: parameter tuning in control pc, change foot position in kinematics model by 1.2

File: RobotSystems/Mercury/mercury.urdf (robot description, URDF)
Before this commit: robot mercury, 23 links, 22 joints
Joints:
- joint abduct_r_to_thigh_r_j: origin xyz=0.0 0.0 -0.03535 rpy=0.01 0.0 0.007 -> xyz=0.0 0.0 -0.03535 rpy=0.0 0.0 0.0
- joint ankle_l: origin xyz=0.0 -0.002 -0.47 rpy=0 0 0 -> xyz=0.012 -0.02 -0.47 rpy=0 0 0
- joint ankle_r: origin xyz=0.0 0.0 -0.47 rpy=0 0 0 -> xyz=0.012 -0.01 -0.47 rpy=0 0 0
- joint fixed_led10: origin xyz=0.0 -0.033 -0.47 rpy=0 0 0 -> xyz=0.0 -0.034 -0.47 rpy=0 0 0
- joint fixed_led3: origin xyz=0.035 -0.0 -0.050 rpy=0 0 0 -> xyz=0.035 -0.01 -0.050 rpy=0 0 0
- joint fixed_led4: origin xyz=0.0 -0.025 -0.47 rpy=0 0 0 -> xyz=0.0 -0.045 -0.47 rpy=0 0 0
- joint fixed_led5: origin xyz=0.0 0.025 -0.47 rpy=0 0 0 -> xyz=0.0 0.005 -0.47 rpy=0 0 0
- joint fixed_led9: origin xyz=0.0 0.017 -0.47 rpy=0 0 0 -> xyz=0.0 0.014 -0.47 rpy=0 0 0
- joint thigh_l_to_knee_l_j: origin xyz=0.0181 0.00 -0.4575 rpy=0 0 0.005 -> xyz=0.0181 -0.01 -0.4575 rpy=0 0 0.005

Commit message: rough terrain test

File: RobotSystems/Mercury/mercury.urdf (robot description, URDF)
Before this commit: robot mercury, 23 links, 22 joints
Joints:
- joint ankle_l: origin xyz=0.012 -0.02 -0.47 rpy=0 0 0 -> xyz=0.005 -0.02 -0.47 rpy=0 0 0
- joint ankle_r: origin xyz=0.012 -0.01 -0.47 rpy=0 0 0 -> xyz=0.005 -0.01 -0.47 rpy=0 0 0
