Commit message: assemble mini cheetah

File: Simulator/SimulationModel/MiniCheetah/mini_cheetah.urdf (robot description, URDF)
Before this commit: robot mini_cheetah, 17 links, 16 joints
Links:
- link abduct_fl: mass 2.1656 -> 0.54; geometry collision mesh filename=meshes/mini_abad.obj; visual mesh filename=meshes/mini_abad.obj
- link abduct_hl: mass 2.1656 -> 0.54; geometry collision mesh filename=meshes/mini_abad.obj; visual mesh filename=meshes/mini_abad.obj
- link abduct_hr: mass 2.1656 -> 0.54; geometry collision mesh filename=meshes/mini_abad.obj; visual mesh filename=meshes/mini_abad.obj
- link foot_fl: geometry collision capsule length=0.12 radius=0.05
- link foot_fr: mass 0.123 -> 0.00001
- link foot_hl: geometry collision capsule length=0.12 radius=0.05
- link foot_hr: geometry collision capsule length=0.12 radius=0.05
- link shank_fl: mass 0.649 -> 0.064; geometry collision mesh filename=meshes/mini_lower_link.obj; visual mesh filename=meshes/mini_lower_link.obj
- link shank_hl: mass 0.649 -> 0.064; geometry collision mesh filename=meshes/mini_lower_link.obj; visual mesh filename=meshes/mini_lower_link.obj
- link shank_hr: mass 0.649 -> 0.064; geometry collision mesh filename=meshes/mini_lower_link.obj; visual mesh filename=meshes/mini_lower_link.obj
- link thigh_fl: mass 3.2 -> 0.634; geometry collision mesh filename=meshes/mini_upper_link.obj; visual mesh filename=meshes/mini_upper_link.obj
- link thigh_hl: mass 3.2 -> 0.634; geometry collision mesh filename=meshes/mini_upper_link.obj; visual mesh filename=meshes/mini_upper_link.obj
- link thigh_hr: mass 3.2 -> 0.634; geometry collision mesh filename=meshes/mini_upper_link.obj; visual mesh filename=meshes/mini_upper_link.obj
Joints:
- joint abduct_fl_to_thigh_fl_j: axis 0 1 0 -> 0 -1 0; origin xyz=0.0 0.02 -0.02 rpy=0.0 0.0 0.0 -> xyz=0.0 0.062 0.00 rpy=0.0 0.0 0.0
- joint abduct_fr_to_thigh_fr_j: axis 0 1 0 -> 0 -1 0
- joint abduct_hl_to_thigh_hl_j: axis 0 1 0 -> 0 -1 0; origin xyz=0.0 0.02 -0.02 rpy=0.0 0.0 0.0 -> xyz=0.0 0.062 0.00 rpy=0.0 0.0 0.0
- joint abduct_hr_to_thigh_hr_j: axis 0 1 0 -> 0 -1 0; origin xyz=0.0 -0.02 -0.02 rpy=0.0 0.0 0.0 -> xyz=0.0 -0.062 0.00 rpy=0.0 0.0 0.0
- joint ankle_fl: origin xyz=0.0 0.0 -0.135 rpy=0 0 0 -> xyz=0.0 0.0 -0.175 rpy=0 0 0
- joint ankle_fr: origin xyz=0.0 0.0 -0.135 rpy=0 0 0 -> xyz=0.0 0.0 -0.175 rpy=0 0 0
- joint ankle_hl: origin xyz=0.0 0.0 -0.135 rpy=0 0 0 -> xyz=0.0 0.0 -0.175 rpy=0 0 0
- joint ankle_hr: origin xyz=0.0 0.0 -0.135 rpy=0 0 0 -> xyz=0.0 0.0 -0.175 rpy=0 0 0
- joint thigh_fl_to_knee_fl_j: axis 0 1 0 -> 0 -1 0; origin xyz=0.0 0.0 -0.15 rpy=0.0 0 0.0 -> xyz=0.0 0.0 -0.209 rpy=0.0 0 0.0
- joint thigh_fr_to_knee_fr_j: axis 0 1 0 -> 0 -1 0; origin xyz=0.0 0.0 -0.15 rpy=0.0 0 0.0 -> xyz=0.0 0.0 -0.209 rpy=0.0 0 0.0
- joint thigh_hl_to_knee_hl_j: axis 0 1 0 -> 0 -1 0; origin xyz=0.0 0.0 -0.15 rpy=0.0 0 0.0 -> xyz=0.0 0.0 -0.209 rpy=0.0 0 0.0
- joint thigh_hr_to_knee_hr_j: axis 0 1 0 -> 0 -1 0; origin xyz=0.0 0.0 -0.15 rpy=0.0 0 0.0 -> xyz=0.0 0.0 -0.209 rpy=0.0 0 0.0
- joint torso_to_abduct_fl_j: origin xyz=0.175 0.1 0.0 rpy=0 0 0 -> xyz=0.19 0.049 0.0 rpy=0 0 0
- joint torso_to_abduct_hl_j: origin xyz=-0.175 0.1 0.0 rpy=0 0 0 -> xyz=-0.19 0.049 0.0 rpy=0 0 0
- joint torso_to_abduct_hr_j: origin xyz=-0.175 -0.1 0.0 rpy=0 0 0 -> xyz=-0.19 -0.049 0.0 rpy=0 0 0
