Commit message: mini cheetah assembly in DART

File: Simulator/SimulationModel/MiniCheetah/mini_cheetah_srlib.urdf (robot description, URDF)
Before this commit: robot mini_cheetah, 13 links, 12 joints
Links:
- added link foot_fl, mass 0.123; collision capsule length=0.12 radius=0.05
- added link foot_fr, mass 0.00001; collision sphere radius=0.03
- added link foot_hl, mass 0.123; collision capsule length=0.12 radius=0.05
- added link foot_hr, mass 0.123; collision capsule length=0.12 radius=0.05
Joints:
- added joint ankle_fl: type fixed, parent shank_fl, child foot_fl, origin xyz=0.0 0.0 -0.175 rpy=0 0 0, axis 0 1 0
- added joint ankle_fr: type fixed, parent shank_fr, child foot_fr, origin xyz=0.0 0.0 -0.175 rpy=0 0 0, axis 0 1 0
- added joint ankle_hl: type fixed, parent shank_hl, child foot_hl, origin xyz=0.0 0.0 -0.175 rpy=0 0 0, axis 0 1 0
- added joint ankle_hr: type fixed, parent shank_hr, child foot_hr, origin xyz=0.0 0.0 -0.175 rpy=0 0 0, axis 0 1 0
